Commit message: feat: establish mulo x-1 ros2 foundation

File: src/rover_description/urdf/axiom_rover.urdf (robot description, URDF)
Before this commit: robot axiom_rover, 2 links, 1 joints
Links:
- removed link winch_drum
- added link base_footprint
- added link camera_link, mass 0.072; visual box size=0.09 0.025 0.025
- added link camera_optical_frame
- added link imu_link, mass 0.05; visual box size=0.04 0.04 0.01
- added link pivot_link, mass 0.5; visual cylinder length=0.06 radius=0.02
- added link wheel_fl_link, mass 4.0; collision cylinder length=0.07 radius=0.254; visual cylinder length=0.07 radius=0.254
- added link wheel_fr_link, mass 4.0; collision cylinder length=0.07 radius=0.254; visual cylinder length=0.07 radius=0.254
- added link wheel_rl_link, mass 4.0; collision cylinder length=0.07 radius=0.254; visual cylinder length=0.07 radius=0.254
- added link wheel_rr_link, mass 4.0; collision cylinder length=0.07 radius=0.254; visual cylinder length=0.07 radius=0.254
- added link winch_drum_link, mass 3.0; collision cylinder length=0.2 radius=0.05; visual cylinder length=0.2 radius=0.05
- link base_link: mass None -> 80.0
Joints:
- added joint base_footprint_joint: type fixed, parent base_footprint, child base_link, origin xyz=0 0 0.254 rpy=0 0 0
- added joint camera_joint: type fixed, parent base_link, child camera_link, origin xyz=0.42 0 0.32 rpy=0 0.26 0
- added joint camera_optical_joint: type fixed, parent camera_link, child camera_optical_frame, origin xyz=0 0 0 rpy=-1.5708 0 -1.5708
- added joint imu_joint: type fixed, parent base_link, child imu_link, origin xyz=0 0 0.31 rpy=0 0 0
- added joint pivot_joint: type revolute, parent base_link, child pivot_link, origin xyz=0 0 0.15 rpy=0 0 0, axis 1 0 0, limit lower=-0.35 upper=0.35 effort=500 velocity=0.5
- added joint wheel_fl_joint: type continuous, parent base_link, child wheel_fl_link, origin xyz=0.35 0.335 0 rpy=0 0 0, axis 0 1 0
- added joint wheel_fr_joint: type continuous, parent base_link, child wheel_fr_link, origin xyz=0.35 -0.335 0 rpy=0 0 0, axis 0 1 0
- added joint wheel_rl_joint: type continuous, parent base_link, child wheel_rl_link, origin xyz=-0.35 0.335 0 rpy=0 0 0, axis 0 1 0
- added joint wheel_rr_joint: type continuous, parent base_link, child wheel_rr_link, origin xyz=-0.35 -0.335 0 rpy=0 0 0, axis 0 1 0
- joint winch_joint: axis 0 0 1 -> 0 1 0; child winch_drum -> winch_drum_link; origin xyz=0.35 0 0.15 rpy=0 1.57 0 -> xyz=0.38 0 0.1 rpy=0 0 0
